File: Passive Mult.brd (EAGLE design)
At the start: 7.6 x 106.7 mm, 11 parts, among them J1 OG-PJ301_PJ301_THONKICONN4, J2 OG-PJ301_PJ301_THONKICONN4, J3 OG-PJ301_PJ301_THONKICONN4, J4 OG-PJ301_PJ301_THONKICONN4, J5 OG-PJ301_PJ301_THONKICONN4, J6 OG-PJ301_PJ301_THONKICONN4, J7 OG-PJ301_PJ301_THONKICONN4, J8 OG-PJ301_PJ301_THONKICONN4

Commit message: BottomSilk updated, front-panel holes and dimension dxf added
Other:
- board text added: "TomaTek 2017"
Changed lines of the file:
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@@
 <?xml version="1.0" encoding="utf-8"?>
 <!DOCTYPE eagle SYSTEM "eagle.dtd">
-<eagle version="7.2.0">
+<eagle version="8.0.0">
 <drawing>
 <settings>
@@
 <layer number="42" name="bRestrict" color="1" fill="10" visible="no" active="yes"/>
 <layer number="43" name="vRestrict" color="2" fill="10" visible="no" active="yes"/>
-<layer number="44" name="Drills" color="7" fill="1" visible="no" active="yes"/>
+<layer number="44" name="Drills" color="7" fill="1" visible="yes" active="yes"/>
 <layer number="45" name="Holes" color="7" fill="1" visible="no" active="yes"/>
 <layer number="46" name="Milling" color="3" fill="1" visible="no" active="yes"/>
@@
 <layer number="110" name="110" color="7" fill="1" visible="no" active="yes"/>
 <layer number="111" name="111" color="7" fill="1" visible="no" active="yes"/>
-<layer number="112" name="tSilk" color="7" fill="1" visible="no" active="yes"/>
+<layer number="112" name="tSilk" color="7" fill="1" visible="yes" active="yes"/>
 <layer number="113" name="bsilk" color="7" fill="1" visible="yes" active="yes"/>
 <layer number="116" name="Patch_BOT" color="7" fill="1" visible="no" active="yes"/>
@@
 <text x="5.08" y="113.665" size="1.016" layer="113" font="vector" rot="MR0" align="bottom-center">top side</text>
 <wire x1="8.255" y1="113.03" x2="1.905" y2="113.03" width="0.3048" layer="113"/>
+<text x="6.985" y="20.955" size="1.4224" layer="113" rot="MR90">TomaTek 2017</text>
 </plain>
 <attributes>
